File: Placa/micro.sch (KiCad schematic (older format))
At the start: 24 parts, among them IC1 ATMEGA16-A, P1 CONN_3X2, P2 CONN_5X2, P3 CONN_5X2, P6 CONN_2, P7 CONN_7X2, P9 CONN_5X2, Q1 NPN, SW1 SW_PUSH, SW2 SW_PUSH, U1 MAX232, X1 8 MHz

Commit message: Agrego cambios en la placa microcontrolador, propuestos por Joaco:
1) Agrego filtro para los AD
2) Agrego resistencias para cada led de los sensores
3) Hice algo mas pero no recuerdo que.
Parts:
- removed P3: CONN_5X2, symbol CONN_5X2
- added C10: 100nF, symbol C
- added C11: C, symbol C
- added L1: INDUCTOR, symbol INDUCTOR
- added P3: CONN_8X2, symbol CONN_8X2
- added R3, R4, R5, R6, R7: R, symbol R
Connections:
- net labels added: S-, S1+, S2+, S3+, S4+, S5+, S6+
- net labels removed: Alimentación_Sensores
- wire segments 121 -> 149
Other:
- moved on the sheet: C3, P6

Commit message: Agrego archivos placa potencia. Agrego biblioteca ptn78020w.
Parts:
- C1: value 22 pF -> 12 pF
- C6: renamed from C11; value C -> 100nF
- L1: value INDUCTOR -> 10uH
- renumbered C7 to C10, C8 to C11, C9 to C3, C3 to C4, C10 to C5, C4 to C7, C5 to C8, C6 to C9, P7 to P1, P1 to P3, P6 to P4, P9 to P5, P3 to P6
Changed lines of the file:
@@
-EESchema Schematic File Version 2  date lun 29 abr 2013 17:14:43 ART
+EESchema Schematic File Version 2  date sáb 25 may 2013 16:00:35 ART
 LIBS:power
 LIBS:device
@@
 LIBS:contrib
 LIBS:valves
+LIBS:cny70
+LIBS:L298
+LIBS:ptn4050
+LIBS:ptn78000w
+LIBS:ptn78020w
+LIBS:TCO-cache
 EELAYER 25  0
 EELAYER END
 $Descr A4 11700 8267
 encoding utf-8
-Sheet 1 1
+Sheet 2 5
 Title "TCO"
-Date "29 apr 2013"
+Date "25 may 2013"
 Rev "1"
 Comp "Club de Robótica de la Facultad de Ingeniería de la Universidad de Buenos Aires"
@@
 Connection ~ 2250 3250
 $Comp
-L C C10
+L C C5
 U 1 1 517EC291
 P 1950 3250
-F 0 "C10" V 2200 3250 50  0000 L CNN
+F 0 "C5" V 2200 3250 50  0000 L CNN
 F 1 "100nF" V 2100 3150 50  0000 L CNN
 	1    1950 3250
@@
 $EndComp
 $Comp
-L C C11
+L C C6
 U 1 1 517EC041
 P 3350 3250
-F 0 "C11" V 3400 3350 50  0000 L CNN
-F 1 "C" V 3400 3150 50  0000 L CNN
+F 0 "C6" V 3400 3350 50  0000 L CNN
+F 1 "100nF" V 3150 3100 50  0000 L CNN
 	1    3350 3250
 	0    -1   -1   0
@@
 P 2750 3250
 F 0 "L1" V 2700 3250 40  0000 C CNN
-F 1 "INDUCTOR" V 2850 3250 40  0000 C CNN
+F 1 "10uH" V 2850 3250 40  0000 C CNN
 	1    2750 3250
 	0    -1   -1   0
@@
 Sensor_Piso_Izq
 $Comp
-L CONN_8X2 P3
+L CONN_8X2 P6
 U 1 1 517EBEA3
 P 9450 1300
-F 0 "P3" H 9450 1750 60  0000 C CNN
+F 0 "P6" H 9450 1750 60  0000 C CNN
 F 1 "CONN_8X2" V 9450 1300 50  0000 C CNN
 	1    9450 1300
@@
 NoConn ~ 8900 2550
 $Comp
-L CONN_5X2 P9
+L CONN_5X2 P5
 U 1 1 517BFEF9
 P 9300 2450
-F 0 "P9" H 9300 2750 60  0000 C CNN
+F 0 "P5" H 9300 2750 60  0000 C CNN
 F 1 "CONN_5X2" V 9300 2450 50  0000 C CNN
 	1    9300 2450
@@
 $EndComp
 $Comp
-L CONN_2 P6
+L CONN_2 P4
 U 1 1 517C1CE8
 P 7950 4300
-F 0 "P6" V 7900 4300 40  0000 C CNN
+F 0 "P4" V 7900 4300 40  0000 C CNN
 F 1 "CONN_2" V 8000 4300 40  0000 C CNN
 	1    7950 4300
@@
 $EndComp
 $Comp
-L C C9
+L C C3
 U 1 1 51746DA2
 P 1450 5100
-F 0 "C9" H 1050 5200 50  0000 L CNN
+F 0 "C3" H 1050 5200 50  0000 L CNN
 F 1 "100nF" H 1050 5100 50  0000 L CNN
 	1    1450 5100
@@
 Motor_1_Direction
 $Comp
-L CONN_7X2 P7
+L CONN_7X2 P1
 U 1 1 517467EE
 P 2100 2350
-F 0 "P7" H 2100 2750 60  0000 C CNN
+F 0 "P1" H 2100 2750 60  0000 C CNN
 F 1 "CONN_7X2" V 2100 2350 50  0000 C CNN
 	1    2100 2350
@@
 $EndComp
 $Comp
-L CAPAPOL C8
+L CAPAPOL C11
 U 1 1 51742251
 P 6500 2150
-F 0 "C8" H 6550 2250 50  0000 L CNN
+F 0 "C11" H 6550 2250 50  0000 L CNN
 F 1 "1uF" H 6550 2050 50  0000 L CNN
 	1    6500 2150
@@
 $EndComp
 $Comp
-L CAPAPOL C6
+L CAPAPOL C9
 U 1 1 5174224C
 P 6200 1650
-F 0 "C6" H 6250 1750 50  0000 L CNN
+F 0 "C9" H 6250 1750 50  0000 L CNN
 F 1 "1uF" H 6250 1550 50  0000 L CNN
 	1    6200 1650
@@
 $EndComp
 $Comp
-L CAPAPOL C7
+L CAPAPOL C10
 U 1 1 51742246
 P 6500 1250
-F 0 "C7" H 6550 1350 50  0000 L CNN
+F 0 "C10" H 6550 1350 50  0000 L CNN
 F 1 "1uF" H 6550 1150 50  0000 L CNN
 	1    6500 1250
@@
 TXD
 $Comp
-L CAPAPOL C5
+L CAPAPOL C8
 U 1 1 51742178
 P 4200 1750
-F 0 "C5" H 3900 1750 50  0000 L CNN
+F 0 "C8" H 3900 1750 50  0000 L CNN
 F 1 "1uF" H 4350 1750 50  0000 L CNN
 	1    4200 1750
@@
 $EndComp
 $Comp
-L CAPAPOL C4
+L CAPAPOL C7
 U 1 1 5174216E
 P 4200 1250
-F 0 "C4" H 3900 1250 50  0000 L CNN
+F 0 "C7" H 3900 1250 50  0000 L CNN
 F 1 "1uF" H 4350 1250 50  0000 L CNN
 	1    4200 1250
@@
 MOSI
 $Comp
-L CONN_3X2 P1
+L CONN_3X2 P3
 U 1 1 51741714
 P 7950 3450
-F 0 "P1" H 7950 3700 50  0000 C CNN
+F 0 "P3" H 7950 3700 50  0000 C CNN
 F 1 "CONN_3X2" V 7950 3500 40  0000 C CNN
 	1    7950 3450
@@
 $EndComp
 $Comp
-L C C3
+L C C4
 U 1 1 5174105F
 P 1550 900
-F 0 "C3" V 1650 1000 50  0000 L CNN
+F 0 "C4" V 1650 1000 50  0000 L CNN
 F 1 "100 nF" V 1750 800 50  0000 L CNN
 	1    1550 900
@@
 P 850 4100
 F 0 "C1" V 700 3900 50  0000 L CNN
-F 1 "22 pF" V 700 4050 50  0000 L CNN
+F 1 "12 pF" V 700 4050 50  0000 L CNN
 	1    850  4100
 	0    1    1    0
