File: Placa/micro.sch (KiCad schematic (older format))
At the start: 32 parts, among them IC1 ATMEGA16-A, P1 CONN_7X2, P2 CONN_5X2, P3 CONN_3X2, P4 CONN_2, P5 CONN_5X2, P6 CONN_8X2, Q1 NPN, SW1 SW_PUSH, SW2 SW_PUSH, U1 MAX232, X1 8 MHz

Commit message: Hice la documentacion para la compentencia. Ademas arregle en el Kicad el reset del micro.
Connections:
- wire segments 149 -> 150
Other:
- moved on the sheet: C4

Commit message: Placa microcontrolador revisión 2. Agrego modificaciones: posibildad de encender todos los sensores desde el micro. Identificar interrupción de cada sensor.
Parts:
- removed 1k1, R2, R3, R4, R5, R6, R7: R, symbol R
- removed P5: CONN_5X2, symbol CONN_5X2
- removed P6: CONN_8X2, symbol CONN_8X2
- removed Q1: NPN, symbol NPN
- added C?: 100nF, symbol C
- added D? (x7): DIODE, symbol DIODE
- added F?: FUSE, symbol FUSE
- added P?: UNL2803A, symbol DIL18
- added P? (x2): CONN_5X2, symbol CONN_5X2
- added R?: R, symbol R
Connections:
- net labels added: Echo_Sensor_Pared_Cen, Echo_Sensor_Pared_Der, Echo_Sensor_Pared_Izq, Encendido_Sens_Pared_Cen, Encendido_Sens_Pared_Der, Encendido_Sens_Pared_Izq, Encendido_Sens_Piso_Cen, Encendido_Sens_Piso_Der, Encendido_Sens_Piso_Izq, Interrupcion_sensores, Led_Test_Rojo, Led_Test_Verde, Micro_Encendido_Sens_Pared, Micro_Encendido_Sens_Piso, Micro_Led_Test_Rojo, Micro_Led_Test_Verde, Trigger_Sensor_Pared_Cen, Trigger_Sensor_Pared_Der, Trigger_Sensor_Pared_Izq
- net labels removed: Encendido_Sensores, INT2, S-, S1+, S2+, S3+, S4+, S5+, S6+, Sensor_Pared_Cen, Sensor_Pared_Der, Sensor_Pared_Izq, Señal_sens_pared, TCK, TDI, TDO, TIMER1, TMS
- wire segments 150 -> 136
- no-connect marks 15 -> 14
Other:
- note added: "Circuito driver para menejar sensores"
- note added: "Conexión sensores pared"
- note added: "Conexión sensores pisos"
- note added: "OR de diodos para la interrupción"
- note removed: "Conexión JTAG"
- note removed: "Conexión sensores"
- note removed: "Encendido sensores"
- note removed: "Switch 1"
- moved on the sheet: C4, P4

Commit message: Me olvidé de agregar los LED's indicadores.
Parts:
- added D? (x2): LED, symbol LED
- added R? (x2): 470, symbol R
- R?: value R -> 10 k
Connections:
- wire segments 136 -> 139
Other:
- note added: "LEDs indicadores"
Changed lines of the file:
@@
-EESchema Schematic File Version 2  date mar 11 jun 2013 15:56:30 ART
+EESchema Schematic File Version 2  date mar 11 jun 2013 16:06:38 ART
 LIBS:power
 LIBS:device
@@
 Comment4 ""
 $EndDescr
+Connection ~ 9900 4150
+Connection ~ 9900 4450
+Wire Wire Line
+	9250 4450 9900 4450
+Connection ~ 10300 4150
+Connection ~ 10300 4450
+Connection ~ 10800 4150
+Connection ~ 10800 4450
+Connection ~ 10800 4550
+Wire Wire Line
+	10800 4150 10800 4550
 Wire Notes Line
 	5200 4700 8600 4700
@@
 Wire Notes Line
 	8600 6900 5200 6900
+Wire Notes Line
+	9150 3800 9150 4650
+Wire Notes Line
+	9150 3800 11150 3800
+Wire Notes Line
+	11150 3800 11150 4650
+Wire Notes Line
+	11150 4650 9150 4650
+Wire Wire Line
+	9250 4150 9900 4150
+$Comp
+L GND #PWR?
+U 1 1 51B77519
+P 10800 4550
+F 0 "#PWR?" H 10800 4550 30  0001 C CNN
+F 1 "GND" H 10800 4480 30  0001 C CNN
+	1    10800 4550
+	1    0    0    -1
+$EndComp
+$Comp
+L R R?
+U 1 1 51B774F4
+P 10550 4450
+F 0 "R?" V 10630 4450 50  0000 C CNN
+F 1 "470" V 10550 4450 50  0000 C CNN
+	1    10550 4450
+	0    -1   -1   0
+$EndComp
+$Comp
+L R R?
+U 1 1 51B774EF
+P 10550 4150
+F 0 "R?" V 10630 4150 50  0000 C CNN
+F 1 "470" V 10550 4150 50  0000 C CNN
+	1    10550 4150
+	0    -1   -1   0
+$EndComp
+$Comp
+L LED D?
+U 1 1 51B774C9
+P 10100 4450
+F 0 "D?" H 10100 4550 50  0000 C CNN
+F 1 "LED" H 10100 4350 50  0000 C CNN
+	1    10100 4450
+	1    0    0    -1
+$EndComp
+$Comp
+L LED D?
+U 1 1 51B774C5
+P 10100 4150
+F 0 "D?" H 10100 4250 50  0000 C CNN
+F 1 "LED" H 10100 4050 50  0000 C CNN
+	1    10100 4150
+	1    0    0    -1
+$EndComp
+Text Label 9250 4450 0    60   ~ 0
+Led_Test_Rojo
+Text Label 9250 4150 0    60   ~ 0
+Led_Test_Verde
+Text Notes 9200 3950 0    60   ~ 0
+LEDs indicadores
 Text Notes 6900 4850 0    60   ~ 0
 OR de diodos para la interrupción
@@
 P 7000 6700
 F 0 "R?" V 7080 6700 50  0000 C CNN
-F 1 "R" V 7000 6700 50  0000 C CNN
+F 1 "10 k" V 7000 6700 50  0000 C CNN
 	1    7000 6700
 	0    -1   -1   0

Commit message: Agrego retoques en 2da revisión PCB micro
Parts:
- X1: value 8 MHz -> 16 MHz
- gave numbers to parts that had none: 17

Commit message: Se agrega PCB placa micros revisión 2.
Parts:
- added R5, R6, R7: 200, symbol R
- C4: value 100 nF -> 10 uF

Commit message: Agrego esquematico versión 1 PCB micro para poder usar de referencia hasta que fabriquemos la segunda placa.
Parts:
- removed C22: 100nF, symbol C
- removed D10, D11, D12, D13, D14, D15, D9: DIODE, symbol DIODE
- removed D16, D17: LED, symbol LED
- removed F1: FUSE, symbol FUSE
- removed P21, P6: CONN_5X2, symbol CONN_5X2
- removed P5: UNL2803A, symbol DIL18
- added 1k1: R, symbol R
- added P3: CONN_8X2, symbol CONN_8X2
- added P9: CONN_5X2, symbol CONN_5X2
- added Q1: NPN, symbol NPN
- C1: value 12 pF -> 22 pF
- C11: renamed from C6; value 100nF -> C
- C3: renamed from C4; value 10 uF -> 100 nF
- L1: value 10uH -> INDUCTOR
- R2: value 10 k -> R
- R3, R4: value 470 -> R
- R5, R6, R7: value 200 -> R
- X1: value 16 MHz -> 8 MHz
- renumbered C5 to C10, C7 to C4, C8 to C5, C9 to C6, C10 to C7, C11 to C8, C3 to C9, P3 to P1, P4 to P6, P1 to P7
Connections:
- net labels added: Encendido_Sensores, INT2, S-, S1+, S2+, S3+, S4+, S5+, S6+, Sensor_Pared_Cen, Sensor_Pared_Der, Sensor_Pared_Izq, Señal_sens_pared, TCK, TDI, TDO, TIMER1, TMS
- net labels removed: Echo_Sensor_Pared_Cen, Echo_Sensor_Pared_Der, Echo_Sensor_Pared_Izq, Encendido_Sens_Pared_Cen, Encendido_Sens_Pared_Der, Encendido_Sens_Pared_Izq, Encendido_Sens_Piso_Cen, Encendido_Sens_Piso_Der, Encendido_Sens_Piso_Izq, Interrupcion_sensores, Led_Test_Rojo, Led_Test_Verde, Micro_Encendido_Sens_Pared, Micro_Encendido_Sens_Piso, Micro_Led_Test_Rojo, Micro_Led_Test_Verde, Trigger_Sensor_Pared_Cen, Trigger_Sensor_Pared_Der, Trigger_Sensor_Pared_Izq
- wire segments 139 -> 150
Other:
- note added: "Conexión JTAG"
- note added: "Conexión sensores"
- note added: "Encendido sensores"
- note added: "Switch 1"
- note removed: "Circuito driver para menejar sensores"
- note removed: "Conexión sensores pared"
- note removed: "Conexión sensores pisos"
- note removed: "LEDs indicadores"
- note removed: "OR de diodos para la interrupción"
- moved on the sheet: C3, P6

Commit message: Se cargaron las versiones correctas de los esquemáticos y los PCB.
Parts:
- C1: value 22 pF -> 12 pF
- C6: renamed from C11; value C -> 100nF
- L1: value INDUCTOR -> 10uH
- renumbered C7 to C10, C8 to C11, C9 to C3, C3 to C4, C10 to C5, C4 to C7, C5 to C8, C6 to C9, P7 to P1, P1 to P3, P6 to P4, P9 to P5, P3 to P6
Connections:
- no-connect marks 14 -> 15
Other:
- moved on the sheet: C4
