File: Placa/alimentacion.sch (KiCad schematic (older format))
At the start: 0 parts

Commit message: Agrego archivos placa potencia. Agrego biblioteca ptn78020w.
Parts:
- added C20, C21: 2,2uF, symbol C
- added C22, C23: 330uF, symbol CAPAPOL
- added D1, D2, D3, D4, D5, D6: DIODE, symbol DIODE
- added D10, D11, D12, D7, D8, D9: LED, symbol LED
- added P11, P12, P13, P19, P20: CONN_2, symbol CONN_2
- added P14, P15, P16: CONN_4, symbol CONN_4
- added P17: CONN_8X2, symbol CONN_8X2
- added P18: CONN_5X2, symbol CONN_5X2
- added R10: 732, symbol R
- added R11, R13, R14, R15, R16: 470, symbol R
- added R12: 1k, symbol R
- added R8: R, symbol R
- added R9: 21k, symbol R
- added SW3: SWITCH_INV, symbol SWITCH_INV
- added U2, U3: PTN78020W, symbol PTN78020W
Connections:
- net labels added: +12V, +5V, +BATT, GND, GND LED sensores, Interrupción sensores, NC, Output sensor pared centro, Output sensor pared derecho, Output sensor pared izquierda, PA0 - Sensor piso izquierda, PA1 - Sensor piso Centro, PA2 - Sensor piso derecha, PA3 - Sensor pared izquierda, PA4 - Sensor pared derecha, PA5 - Sensor pared centro, Vcc sensor piso centro, Vcc sensor piso derecha, Vcc sensor piso izquierda
- wire segments 0 -> 90
- no-connect marks 0 -> 6
Other:
- note added: "Conector baterías y switch encendido/apagado"
- note added: "Conector desde la placa de potencia hacia la placa con los CNY70"
- note added: "Conector sensores pared"
- note added: "Fuente DC/DC"
- note added: "Interrupciones"
- note added: "Nota: C20 y C21 son cerámicos"
- note added: "Placa para conectar la placa de potencia con la placa del micro"

Commit message: Agrego alimentación.brd, placa donde se va a montar motores/sensores/baterías.
Parts:
- removed C22: 330uF, symbol CAPAPOL
- removed D10, D11, D12, D9: LED, symbol LED
- removed R13, R14, R15, R16: 470, symbol R
- removed U2: PTN78020W, symbol PTN78020W
- added C25: 100uF, symbol CAPAPOL
- added U2: PTN78000W, symbol PTN78000W
- R11: value 470 -> 21 k
- R12: value 1k -> R
- R9: value 21k -> R
Connections:
- net labels removed: NC
- wire segments 90 -> 94
Other:
- moved on the sheet: P19, P20

Commit message: Agrego retoques en 2da revisión PCB micro
Parts:
- removed D1, D2, D3, D4, D5, D6: DIODE, symbol DIODE
- removed D7, D8: LED, symbol LED
- removed P17: CONN_8X2, symbol CONN_8X2
- removed P18: CONN_5X2, symbol CONN_5X2
- removed R12, R8, R9: R, symbol R
- added P17: CONN_5X2, symbol CONN_5X2
Connections:
- net labels added: Echo_Sens_Pared_Cen, Echo_Sens_Pared_Der, Echo_Sens_Pared_Izq, Encendido_Sens_Pared_Cen, Encendido_Sens_Pared_Der, Encendido_Sens_Pared_Izq, Trigger_Sens_Pared_Cen, Trigger_Sens_Pared_Der, Trigger_Sens_Pared_Izq
- net labels removed: GND LED sensores, Interrupción sensores, Output sensor pared centro, Output sensor pared derecho, Output sensor pared izquierda, PA0 - Sensor piso izquierda, PA1 - Sensor piso Centro, PA2 - Sensor piso derecha, PA3 - Sensor pared izquierda, PA4 - Sensor pared derecha, PA5 - Sensor pared centro, Vcc sensor piso centro, Vcc sensor piso derecha, Vcc sensor piso izquierda
- wire segments 94 -> 52
- no-connect marks 6 -> 3
Other:
- note removed: "Conector desde la placa de potencia hacia la placa con los CNY70"
- note removed: "Interrupciones"
- note removed: "Placa para conectar la placa de potencia con la placa del micro"
- moved on the sheet: C20, C21, C23, C25, P19, P20

Commit message: Se cargaron las versiones correctas de los esquemáticos y los PCB.
Parts:
- removed P17: CONN_5X2, symbol CONN_5X2
- added D1, D2, D3, D4, D5, D6: DIODE, symbol DIODE
- added D7, D8: LED, symbol LED
- added P17: CONN_8X2, symbol CONN_8X2
- added P18: CONN_5X2, symbol CONN_5X2
- added R12, R8, R9: R, symbol R
Connections:
- net labels added: GND LED sensores, Interrupción sensores, Output sensor pared centro, Output sensor pared derecho, Output sensor pared izquierda, PA0 - Sensor piso izquierda, PA1 - Sensor piso Centro, PA2 - Sensor piso derecha, PA3 - Sensor pared izquierda, PA4 - Sensor pared derecha, PA5 - Sensor pared centro, Vcc sensor piso centro, Vcc sensor piso derecha, Vcc sensor piso izquierda
- net labels removed: Echo_Sens_Pared_Cen, Echo_Sens_Pared_Der, Echo_Sens_Pared_Izq, Encendido_Sens_Pared_Cen, Encendido_Sens_Pared_Der, Encendido_Sens_Pared_Izq, Trigger_Sens_Pared_Cen, Trigger_Sens_Pared_Der, Trigger_Sens_Pared_Izq
- wire segments 52 -> 94
- no-connect marks 3 -> 6
Other:
- note added: "Conector desde la placa de potencia hacia la placa con los CNY70"
- note added: "Interrupciones"
- note added: "Placa para conectar la placa de potencia con la placa del micro"
- moved on the sheet: C20, C21, C23, C25, P19, P20
